File: Board/esp_32_board.kicad_pcb (KiCad board)
At the start: 2 copper layers, 72.5 x 36 mm, 24 parts, among them J1 USB_C_Receptacle_USB2.0_16P, J2 UART, J3 JTAG, J4 Conn_01x06_Pin, J5 Conn_01x06_Pin, J6 Conn_01x06_Pin, J8 Conn_01x06_Pin, SW2 RESET, SW3 SW_Push, U2 USBLC6-2SC6, U4 AMS1117-3.3, U5 ESP32-S3-WROOM-1

Commit message: alot of work
Parts:
- added G***: LOGO, Drawings:githubqr_reszed, F.Cu at (139.5, 129.2)
- added G***: LOGO, Drawings:mycat, F.Cu at (136.8, 103.0)
- moved U5 0.31 mm to (189.4, 118.2)
Other:
- board text added: "github"
