File: Board/esp_32_board.kicad_pcb (KiCad board)
At the start: 2 copper layers, 72.5 x 36 mm, 26 parts, among them J1 USB_C_Receptacle_USB2.0_16P, J2 UART, J3 JTAG, J4 Conn_01x06_Pin, J5 Conn_01x06_Pin, J6 Conn_01x06_Pin, J8 Conn_01x06_Pin, SW2 RESET, SW3 SW_Push, U2 USBLC6-2SC6, U4 AMS1117-3.3, U5 ESP32-S3-WROOM-1

Commit message: work
Routing:
- net Net-(U5-EN): track 42.9 -> 50.8 mm
- net /IO11: track 17.6 -> 16.5 mm
- net VBUS: track 73.1 -> 74.1 mm
- net /IO10: track 20.4 -> 19.5 mm
- net /IO9: track 23.2 -> 22.6 mm
- net +3.3V: track 67.1 -> 67.6 mm, vias 0 -> 1
- net GND: vias 12 -> 26
