File: Board/esp_32_board.kicad_pcb (KiCad board)
At the start: 2 copper layers, 72.5 x 36 mm, 26 parts, among them J1 USB_C_Receptacle_USB2.0_16P, J2 UART, J3 JTAG, J4 Conn_01x06_Pin, J5 Conn_01x06_Pin, J6 Conn_01x06_Pin, J8 Conn_01x06_Pin, SW2 RESET, SW3 SW_Push, U2 USBLC6-2SC6, U4 AMS1117-3.3, U5 ESP32-S3-WROOM-1

Commit message: BOM update
Parts:
- C1(Tantalum)1, C1(Tantalum)2, C9: footprint Capacitor_Tantalum_SMD:CP_EIA-3216-18_Kemet-A_HandSolder -> Capacitor_SMD:C_0805_2012Metric_Pad1.18x1.45mm_HandSolder
Routing:
- net VBUS: track 74.1 -> 73.3 mm

Commit message: Fixed the BOM link issue
Parts:
- C1(Tantalum)1, C1(Tantalum)2, C9: footprint Capacitor_SMD:C_0805_2012Metric_Pad1.18x1.45mm_HandSolder -> Capacitor_Tantalum_SMD:CP_EIA-3216-18_Kemet-A_HandSolder
Routing:
- net VBUS: track 73.3 -> 74.1 mm
