File: Board/esp_32_board.kicad_sch (KiCad schematic)
At the start: 24 parts, among them J1 USB_C_Receptacle_USB2.0_16P, J2 UART, J3 JTAG, J4 Conn_01x06_Pin, J5 Conn_01x06_Pin, J6 Conn_01x06_Pin, J8 Conn_01x06_Pin, SW2 RESET, SW3 SW_Push, U2 USBLC6-2SC6, U4 AMS1117-3.3, U5 ESP32-S3-WROOM-1

Commit message: alot of work
Other:
- title: (none) -> ESP32 Custom Board
Changed lines of the file:
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@@
 	(generator_version "10.0")
 	(paper "A4")
+	(title_block
+		(title "ESP32 Custom Board")
+		(date "2026-10-10")
+		(rev "REV1 ")
+	)
 	(rectangle
 		(start 122.555 12.7)
@@
 		)
 		(property "Value" "PWR_FLAG"
-			(at 20.32 162.56 0)
+			(at 21.59 162.814 0)
 			(show_name no)
 			(do_not_autoplace no)
